File: kicad/scrollwheel_peripheral.kicad_pcb (KiCad board)
At the start: 2 copper layers, 71.5 x 38 mm, 9 parts, among them J1 Conn_01x14_Socket, J2 Conn_01x14_Socket, J3 Conn_01x05_Socket

Commit message: Misc changes
Parts:
- added M3: MountingHole_3.2mm_M3, MountingHole:MountingHole_3.2mm_M3, F.Cu at (114.5, 60.5)
- added M3: MountingHole_3.2mm_M3, MountingHole:MountingHole_3.2mm_M3, F.Cu at (46.5, 59.0)
- added M3: MountingHole_3.2mm_M3, MountingHole:MountingHole_3.2mm_M3, F.Cu at (114.5, 86.0)
- added M3: MountingHole_3.2mm_M3, MountingHole:MountingHole_3.2mm_M3, F.Cu at (67.0, 85.0)
- moved C1 9.50 mm to (49.0, 85.5)
- moved C2 9.50 mm to (53.0, 85.5)
- moved VR1 9.50 mm to (49.3, 67.5)
Routing:
- net GND: track 100.6 -> 0.71 mm
- net Net-(J1-Pin_8): track 48.5 -> 58.0 mm
- net Net-(J1-Pin_6): track 49.0 -> 57.6 mm
- net Net-(J1-Pin_9): track 53.9 -> 62.3 mm
- net Net-(J1-Pin_11): track 26.6 -> 30.7 mm
- removed copper zone on B.Cu, net GND
- removed copper zone on F.Cu, net GND
Other:
- board size 71.5 x 38 mm -> 80 x 37 mm
- board text added: "uwusynth scrollwheel peripheral v0.1"

Commit message: Misc
Parts:
- moved J1 31.5 mm to (73.5, 55.5)
- moved J2 31.5 mm to (88.5, 55.5)
- moved J3 31.5 mm to (75.9, 55.5)
- moved C3 29.9 mm to (109.5, 81.5)
- moved C4 29.9 mm to (114.0, 81.5)
- moved VR2 29.9 mm to (110.1, 63.5)
- moved M3 21.1 mm to (46.0, 86.5), turned to -90 degrees
- moved M3 5.32 mm to (118.5, 57.0), turned to -90 degrees
- moved C1 4.51 mm to (48.6, 81.0)
- moved C2 4.51 mm to (52.7, 81.0)
- moved VR1 4.51 mm to (49.0, 63.0)
- moved M3 4.03 mm to (118.5, 86.5), turned to 90 degrees
- moved M3 1.80 mm to (45.5, 57.5), turned to -90 degrees
Routing:
- net Net-(J1-Pin_9): track 62.3 -> 0.00 mm
- net Net-(J1-Pin_8): track 58.0 -> 0.00 mm
- net Net-(J1-Pin_6): track 57.6 -> 0.00 mm
- net Net-(J1-Pin_11): track 30.7 -> 0.00 mm
- net Net-(J1-Pin_7): track 25.8 -> 0.00 mm
- net Net-(J1-Pin_10): track 24.6 -> 0.00 mm
- net GND: track 0.71 -> 0.00 mm
Other:
- board text added: "uhsynth scrollwheel peripheral v0.1"
- board text removed: "uwusynth scrollwheel peripheral v0.1"

Commit message: footprints
Parts:
- added C10: C, Capacitor_SMD:C_0805_2012Metric, F.Cu at (60.6, 31.3)
- added C11: C, Capacitor_SMD:C_0805_2012Metric, F.Cu at (60.6, 34.3)
- added C5: 0.1uF, Capacitor_SMD:C_0805_2012Metric, F.Cu at (60.6, 16.3)
- added C6: 12pF, Capacitor_SMD:C_0805_2012Metric, F.Cu at (60.6, 19.3)
- added C7: 12pF, Capacitor_SMD:C_0805_2012Metric, F.Cu at (60.6, 22.3)
- added C8: C, Capacitor_SMD:C_0805_2012Metric, F.Cu at (60.6, 25.3)
- added C9: C, Capacitor_SMD:C_0805_2012Metric, F.Cu at (60.6, 28.3)
- added IC1: ATMEGA32U4-AU, project_footprints:QFP80P1200X1200X120-44N, F.Cu at (70.1, 39.1)
- added R1: 22, Resistor_SMD:R_0805_2012Metric, F.Cu at (94.3, 16.3)
- added R2: 22, Resistor_SMD:R_0805_2012Metric, F.Cu at (94.3, 19.2)
- added R3: 5.1, Resistor_SMD:R_0805_2012Metric, F.Cu at (94.3, 22.2)
- added R4: 5.1, Resistor_SMD:R_0805_2012Metric, F.Cu at (94.3, 25.1)
- added R5: 10k, Resistor_SMD:R_0805_2012Metric, F.Cu at (94.3, 28.1)
- added SW1: SW_Push_Dual, Button_Switch_SMD:SW_DIP_SPSTx02_Slide_9.78x7.26mm_W8.61mm_P2.54mm, F.Cu at (88.2, 47.2)
- added Y1: Crystal, Crystal:Crystal_DS26_D2.0mm_L6.0mm_Horizontal, F.Cu at (78.7, 44.1)
- J1: value Conn_01x14_Socket -> UJ20-C-H-G-MSMT-4-P16-TR; footprint Connector_PinSocket_2.54mm:PinSocket_1x14_P2.54mm_Vertical -> project_footprints:UJ20CHGMSMT4P16TR
- J2: value Conn_01x14_Socket -> AVR-JTAG-10; footprint Connector_PinSocket_2.54mm:PinSocket_1x14_P2.54mm_Vertical -> project_footprints:TSW-110-XX-YY-D
- J3: value Conn_01x05_Socket -> TSW-110-07-F-D; footprint Connector_PinSocket_2.54mm:PinSocket_1x05_P2.54mm_Vertical -> project_footprints:TSW-110-XX-YY-D
- moved J2 59.9 mm to (144.8, 35.0)
- moved J3 59.1 mm to (17.9, 44.0), turned to 0 degrees
- moved J1 21.7 mm to (85.7, 37.6)
Connections:
- C1 pad 1: Net-(J1-Pin_9) -> Net-(IC1-(INT.6/AIN0)_PE6)
- C2 pad 1: Net-(J1-Pin_8) -> Net-(IC1-PB5_(PCINT5/OC1A/~{OC4B}/ADC))
- C3 pad 1: Net-(J1-Pin_11) -> Net-(IC1-(SDA/INT1)_PD1)
- C4 pad 1: Net-(J1-Pin_10) -> Net-(VR2-B)
- J1 pad 2: GND -> unconnected-(J1-MH2-Pad2)
- J2 pad 1: unconnected-(J2-Pin_1-Pad1) -> Net-(IC1-PF4_(ADC4/TCK))
- J2 pad 10: unconnected-(J2-Pin_10-Pad10) -> GND
- J2 pad 11: unconnected-(J2-Pin_11-Pad11) -> (no net)
- J2 pad 12: unconnected-(J2-Pin_12-Pad12) -> (no net)
- J2 pad 13: unconnected-(J2-Pin_13-Pad13) -> (no net)
- J2 pad 14: unconnected-(J2-Pin_14-Pad14) -> (no net)
- J2 pad 2: unconnected-(J2-Pin_2-Pad2) -> GND
- J2 pad 3: unconnected-(J2-Pin_3-Pad3) -> Net-(IC1-PF6_(ADC6/TDO))
- J2 pad 4: unconnected-(J2-Pin_4-Pad4) -> /5V
- J2 pad 5: unconnected-(J2-Pin_5-Pad5) -> Net-(IC1-PF5_(ADC5/TMS))
- J2 pad 6: unconnected-(J2-Pin_6-Pad6) -> Net-(IC1-~{RESET})
- J2 pad 7: unconnected-(J2-Pin_7-Pad7) -> /5V
- J2 pad 9: unconnected-(J2-Pin_9-Pad9) -> Net-(IC1-PF7_(ADC7/TDI))
- J3 pad 1: unconnected-(J3-Pin_1-Pad1) -> Net-(IC1-PE2_(~{HWB}))
- J3 pad 3: unconnected-(J3-Pin_3-Pad3) -> Net-(IC1-PC7_(ICP3/CLK0/OC)4A)
- J3 pad 5: unconnected-(J3-Pin_5-Pad5) -> Net-(IC1-PC6_(OC3A/~{OC4A}))
- VR1 pad 1: Net-(J1-Pin_6) -> Net-(IC1-(PCINT7/OC0A/OC1C/~{RTS})_PB7)
- VR1 pad A1: Net-(J1-Pin_9) -> Net-(IC1-(INT.6/AIN0)_PE6)
- VR1 pad B1: Net-(J1-Pin_8) -> Net-(IC1-PB5_(PCINT5/OC1A/~{OC4B}/ADC))
- VR2 pad 1: Net-(J1-Pin_7) -> Net-(IC1-PB6_(PCINT6/OC1B/OC4B/ADC))
- VR2 pad A1: Net-(J1-Pin_11) -> Net-(IC1-(SDA/INT1)_PD1)
- VR2 pad B1: Net-(J1-Pin_10) -> Net-(VR2-B)

Commit message: Part selection; Board
Parts:
- C1, C10, C11, C2, C3, C4, C5, C8, C9, R3, R4: moved to B.Cu
- C6, C7: value 12pF -> 22pF
- J2: footprint project_footprints:TSW-110-XX-YY-D -> Connector_PinHeader_2.54mm:PinHeader_2x05_P2.54mm_Vertical
- SW1: footprint Button_Switch_SMD:SW_DIP_SPSTx02_Slide_9.78x7.26mm_W8.61mm_P2.54mm -> Button_Switch_THT:SW_PUSH_6mm
- Y1: footprint Crystal:Crystal_DS26_D2.0mm_L6.0mm_Horizontal -> Crystal:Crystal_SMD_Abracon_ABM3-2Pin_5.0x3.2mm
- moved R3 65.0 mm to (85.4, 86.6), turned to -90 degrees
- moved R4 63.0 mm to (80.9, 86.7), turned to 90 degrees
- moved R1 62.1 mm to (92.2, 78.3), turned to 90 degrees
- moved J3 62.0 mm to (66.6, 82.4), turned to 90 degrees
- moved R2 59.3 mm to (89.4, 78.3), turned to 90 degrees
- moved C5 58.6 mm to (84.8, 69.6), turned to 180 degrees
- moved J2 57.4 mm to (99.5, 70.3), turned to 180 degrees
- moved C8 52.6 mm to (84.8, 72.0)
- moved C10 50.1 mm to (77.5, 78.4), turned to -90 degrees
- moved R5 48.8 mm to (95.7, 76.8), turned to -90 degrees
- moved J1 48.3 mm to (83.4, 85.8)
- moved C6 47.5 mm to (89.2, 57.2)
- moved C9 45.7 mm to (84.7, 67.2), turned to 180 degrees
- moved SW1 42.8 mm to (102.2, 87.7), turned to 180 degrees
- moved C7 39.4 mm to (78.2, 57.5), turned to 180 degrees
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Connections:
- C7 pad 1: Net-(IC1-(OC0B/SCL/INT0)_PD0) -> Net-(IC1-XTAL1)
- IC1 pad 17: Net-(IC1-(OC0B/SCL/INT0)_PD0) -> Net-(IC1-XTAL1)
- J1 pad A6: Net-(IC1-~{RESET}) -> Net-(J1-DP1)
- J1 pad A7: Net-(IC1-~{RESET}) -> Net-(J1-DN1)
- R1 pad 1: Net-(IC1-~{RESET}) -> Net-(J1-DN1)
- R2 pad 1: Net-(IC1-~{RESET}) -> Net-(J1-DP1)
- Y1 pad 2: Net-(IC1-(OC0B/SCL/INT0)_PD0) -> Net-(IC1-XTAL1)
Routing:
- net /5V: track 0.00 -> 59.6 mm, vias 0 -> 4
- net Net-(IC1-~{RESET}): track 0.00 -> 38.8 mm
- net Net-(IC1-PE2_(~{HWB})): track 0.00 -> 14.6 mm
- net Net-(IC1-PC7_(ICP3/CLK0/OC)4A): track 0.00 -> 13.9 mm
- net Net-(J1-DN1): track 0.00 -> 10.2 mm
- net Net-(IC1-D+): track 0.00 -> 9.14 mm, vias 0 -> 2
- net Net-(J1-DP1): track 0.00 -> 7.98 mm
- net Net-(IC1-D-): track 0.00 -> 7.31 mm
- net Net-(J1-CC1): track 0.00 -> 4.07 mm, vias 0 -> 1
- net Net-(J1-CC2): track 0.00 -> 3.74 mm, vias 0 -> 1
- net Net-(IC1-UCAP): track 0.00 -> 3.37 mm, vias 0 -> 1

Commit message: More routing
Parts:
- R3, R4: moved to F.Cu
- moved R3 12.6 mm to (72.8, 87.1), turned to 180 degrees
- moved R4 8.52 mm to (72.8, 84.2), turned to 0 degrees
- moved R2 6.12 mm to (93.8, 74.1), turned to 180 degrees
- moved R5 5.00 mm to (100.7, 76.7)
- moved R1 2.42 mm to (93.8, 76.5), turned to 180 degrees
Routing:
- net Net-(IC1-~{RESET}): track 38.8 -> 0.00 mm
- net Net-(J1-CC2): track 3.74 -> 13.9 mm, vias 1 -> 0
- net Net-(J1-DP1): track 7.98 -> 16.8 mm
- net Net-(J1-CC1): track 4.07 -> 10.1 mm, vias 1 -> 0
- net Net-(J1-DN1): track 10.2 -> 14.9 mm
- net Net-(IC1-D+): track 9.14 -> 5.15 mm, vias 2 -> 0
- net /5V: track 59.6 -> 58.7 mm, vias 4 -> 6
- net Net-(IC1-D-): track 7.31 -> 6.76 mm

Commit message: Moving stuff
Parts:
- C10: moved to F.Cu
- moved C10 3.02 mm to (74.5, 78.1), turned to 180 degrees
Routing:
- net /5V: track 58.7 -> 60.1 mm, vias 6 -> 5
Changed lines of the file:
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@@
+	)
+	(footprint "Capacitor_SMD:C_0805_2012Metric"
+		(layer "F.Cu")
+		(at 74.525 78.075 180)
+		(descr "Capacitor SMD 0805 (2012 Metric), square (rectangular) end terminal, IPC_7351 nominal, (Body size source: IPC-SM-782 page 76, https://www.pcb-3d.com/wordpress/wp-content/uploads/ipc-sm-782a_amendment_1_and_2.pdf, https://docs.google.com/spreadsheets/d/1BsfQQcO9C6DZCsRaXUlFlo91Tg2WpOkGARC1WS5S8t0/edit?usp=sharing), generated with kicad-footprint-generator")
+		(tags "capacitor")
+		(property "Reference" "C10"
+			(at 0 -1.68 0)
+			(layer "F.SilkS")
+			(effects
+				(font
+					(size 1 1)
+					(thickness 0.15)
+				)
+			)
+		)
+		(property "Value" "C"
+			(at 0 1.68 0)
+			(layer "F.Fab")
+			(effects
+				(font
+					(size 1 1)
+					(thickness 0.15)
+				)
+			)
+		)
+		(property "Datasheet" ""
+			(at 0 0 180)
+			(unlocked yes)
+			(layer "F.Fab")
+			(hide yes)
+			(effects
+				(font
+					(size 1.27 1.27)
+					(thickness 0.15)
+				)
+			)
+		)
+		(property "Description" "Unpolarized capacitor"
+			(at 0 0 180)
+			(unlocked yes)
+			(layer "F.Fab")
+			(hide yes)
+			(effects
+				(font
+					(size 1.27 1.27)
+					(thickness 0.15)
+				)
+			)
+		)
+		(property ki_fp_filters "C_*")
+		(sheetname "/")
+		(sheetfile "scrollwheel_peripheral.kicad_sch")
+		(attr smd)
+		(fp_line
+			(start -0.261252 0.735)
+			(end 0.261252 0.735)
+			(stroke
+				(width 0.12)
+				(type solid)
+			)
+			(layer "F.SilkS")
+		)
+		(fp_line
+			(start -0.261252 -0.735)
+			(end 0.261252 -0.735)
+			(stroke
+				(width 0.12)
+				(type solid)
+			)
+			(layer "F.SilkS")
+		)
+		(fp_line
+			(start 1.7 0.98)
+			(end -1.7 0.98)
+			(stroke
+				(width 0.05)
+				(type solid)
+			)
+			(layer "F.CrtYd")
+		)
+		(fp_line
+			(start 1.7 -0.98)
+			(end 1.7 0.98)
+			(stroke
+				(width 0.05)
+				(type solid)
+			)
+			(layer "F.CrtYd")
+		)
+		(fp_line
+			(start -1.7 0.98)
+			(end -1.7 -0.98)
+			(stroke
+				(width 0.05)
+				(type solid)
+			)
+			(layer "F.CrtYd")
+		)
+		(fp_line
+			(start -1.7 -0.98)
+			(end 1.7 -0.98)
+			(stroke
+				(width 0.05)
+				(type solid)
+			)
+			(layer "F.CrtYd")
+		)
+		(fp_line
+			(start 1 0.625)
+			(end -1 0.625)
+			(stroke
+				(width 0.1)
+				(type solid)
+			)
+			(layer "F.Fab")
+		)
+		(fp_line
+			(start 1 -0.625)
+			(end 1 0.625)
+			(stroke
+				(width 0.1)
+				(type solid)
+			)
+			(layer "F.Fab")
+		)
+		(fp_line
+			(start -1 0.625)
+			(end -1 -0.625)
+			(stroke
+				(width 0.1)
+				(type solid)
+			)
+			(layer "F.Fab")
+		)
+		(fp_line
+			(start -1 -0.625)
+			(end 1 -0.625)
+			(stroke
+				(width 0.1)
+				(type solid)
+			)
+			(layer "F.Fab")
+		)
+		(fp_text user "${REFERENCE}"
+			(at 0 0 0)
+			(layer "F.Fab")
+			(effects
+				(font
+					(size 0.5 0.5)
+					(thickness 0.08)
+				)
+			)
+		)
+		(pad "1" smd roundrect
+			(at -0.95 0 180)
+			(size 1 1.45)
+			(layers "F.Cu" "F.Mask" "F.Paste")
+			(roundrect_rratio 0.25)
+			(net 13 "/5V")
+			(pintype "passive")
+		)
+		(pad "2" smd roundrect
+			(at 0.95 0 180)
+			(size 1 1.45)
+			(layers "F.Cu" "F.Mask" "F.Paste")
+			(roundrect_rratio 0.25)
+			(net 1 "GND")
+			(pintype "passive")
+		)
+		(embedded_fonts no)
+		(model "${KICAD9_3DMODEL_DIR}/Capacitor_SMD.3dshapes/C_0805_2012Metric.wrl"
+			(offset
+				(xyz 0 0 0)
+			)
+			(scale
+				(xyz 1 1 1)
+			)
+			(rotate
+				(xyz 0 0 0)
+			)
+		)
 	)
 	(footprint "Capacitor_SMD:C_0805_2012Metric"
@@
 		(pad "2" smd roundrect
 			(at 0.95 0 180)
-			(size 1 1.45)
-			(layers "B.Cu" "B.Mask" "B.Paste")
-			(roundrect_rratio 0.25)
-			(net 1 "GND")
-			(pintype "passive")
-		)
-		(embedded_fonts no)
-		(model "${KICAD9_3DMODEL_DIR}/Capacitor_SMD.3dshapes/C_0805_2012Metric.wrl"
-			(offset
-				(xyz 0 0 0)
-			)
-			(scale
-				(xyz 1 1 1)
-			)
-			(rotate
-				(xyz 0 0 0)
-			)
-		)
-	)
-	(footprint "Capacitor_SMD:C_0805_2012Metric"
-		(layer "B.Cu")
-		(at 77.525 78.425 -90)
-		(descr "Capacitor SMD 0805 (2012 Metric), square (rectangular) end terminal, IPC_7351 nominal, (Body size source: IPC-SM-782 page 76, https://www.pcb-3d.com/wordpress/wp-content/uploads/ipc-sm-782a_amendment_1_and_2.pdf, https://docs.google.com/spreadsheets/d/1BsfQQcO9C6DZCsRaXUlFlo91Tg2WpOkGARC1WS5S8t0/edit?usp=sharing), generated with kicad-footprint-generator")
-		(tags "capacitor")
-		(property "Reference" "C10"
-			(at 0 1.68 90)
-			(layer "B.SilkS")
-			(effects
-				(font
-					(size 1 1)
-					(thickness 0.15)
-				)
-				(justify mirror)
-			)
-		)
-		(property "Value" "C"
-			(at 0 -1.68 90)
-			(layer "B.Fab")
-			(effects
-				(font
-					(size 1 1)
-					(thickness 0.15)
-				)
-				(justify mirror)
-			)
-		)
-		(property "Datasheet" ""
-			(at 0 0 90)
-			(unlocked yes)
-			(layer "B.Fab")
-			(hide yes)
-			(effects
-				(font
-					(size 1.27 1.27)
-					(thickness 0.15)
-				)
-				(justify mirror)
-			)
-		)
-		(property "Description" "Unpolarized capacitor"
-			(at 0 0 90)
-			(unlocked yes)
-			(layer "B.Fab")
-			(hide yes)
-			(effects
-				(font
-					(size 1.27 1.27)
-					(thickness 0.15)
-				)
-				(justify mirror)
-			)
-		)
-		(property ki_fp_filters "C_*")
-		(sheetname "/")
-		(sheetfile "scrollwheel_peripheral.kicad_sch")
-		(attr smd)
-		(fp_line
-			(start -0.261252 0.735)
-			(end 0.261252 0.735)
-			(stroke
-				(width 0.12)
-				(type solid)
-			)
-			(layer "B.SilkS")
-		)
-		(fp_line
-			(start -0.261252 -0.735)
-			(end 0.261252 -0.735)
-			(stroke
-				(width 0.12)
-				(type solid)
-			)
-			(layer "B.SilkS")
-		)
-		(fp_line
-			(start -1.7 0.98)
-			(end 1.7 0.98)
-			(stroke
-				(width 0.05)
-				(type solid)
-			)
-			(layer "B.CrtYd")
-		)
-		(fp_line
-			(start 1.7 0.98)
-			(end 1.7 -0.98)
-			(stroke
-				(width 0.05)
-				(type solid)
-			)
-			(layer "B.CrtYd")
-		)
-		(fp_line
-			(start -1.7 -0.98)
-			(end -1.7 0.98)
-			(stroke
-				(width 0.05)
-				(type solid)
-			)
-			(layer "B.CrtYd")
-		)
-		(fp_line
-			(start 1.7 -0.98)
-			(end -1.7 -0.98)
-			(stroke
-				(width 0.05)
-				(type solid)
-			)
-			(layer "B.CrtYd")
-		)
-		(fp_line
-			(start -1 0.625)
-			(end 1 0.625)
-			(stroke
-				(width 0.1)
-				(type solid)
-			)
-			(layer "B.Fab")
-		)
-		(fp_line
-			(start 1 0.625)
-			(end 1 -0.625)
-			(stroke
-				(width 0.1)
-				(type solid)
-			)
-			(layer "B.Fab")
-		)
-		(fp_line
-			(start -1 -0.625)
-			(end -1 0.625)
-			(stroke
-				(width 0.1)
-				(type solid)
-			)
-			(layer "B.Fab")
-		)
-		(fp_line
-			(start 1 -0.625)
-			(end -1 -0.625)
-			(stroke
-				(width 0.1)
-				(type solid)
-			)
-			(layer "B.Fab")
-		)
-		(fp_text user "${REFERENCE}"
-			(at 0 0 90)
-			(layer "B.Fab")
-			(effects
-				(font
-					(size 0.5 0.5)
-					(thickness 0.08)
-				)
-				(justify mirror)
-			)
-		)
-		(pad "1" smd roundrect
-			(at -0.95 0 270)
-			(size 1 1.45)
-			(layers "B.Cu" "B.Mask" "B.Paste")
-			(roundrect_rratio 0.25)
-			(net 13 "/5V")
-			(pintype "passive")
-		)
-		(pad "2" smd roundrect
-			(at 0.95 0 270)
 			(size 1 1.45)
 			(layers "B.Cu" "B.Mask" "B.Paste")
@@
 	)
 	(segment
+		(start 75.475 78.075)
+		(end 78.3 75.25)
+		(width 0.2)
+		(layer "F.Cu")
+		(net 13)
+	)
+	(segment
 		(start 85.65 63.75)
 		(end 85.65 65.625)
@@
 	)
 	(segment
-		(start 78.125 75.25)
-		(end 77.575 75.8)
-		(width 0.2)
-		(layer "F.Cu")
-		(net 13)
-	)
-	(segment
 		(start 85.65 67.225057)
 		(end 87.124943 68.7)
@@
 	)
 	(segment
-		(start 79.25 75.25)
-		(end 78.125 75.25)
-		(width 0.2)
-		(layer "F.Cu")
-		(net 13)
-	)
-	(segment
 		(start 87.075 72.575)
 		(end 88.875 72.575)
@@
 	(segment
 		(start 79.25 74.3)
+		(end 79.25 75.25)
+		(width 0.2)
+		(layer "F.Cu")
+		(net 13)
+	)
+	(segment
+		(start 78.3 75.25)
 		(end 79.25 75.25)
 		(width 0.2)
@@
 	)
 	(via
-		(at 77.575 75.8)
-		(size 0.6)
-		(drill 0.3)
-		(layers "F.Cu" "B.Cu")
-		(net 13)
-	)
-	(via
 		(at 87.075 72.575)
 		(size 0.6)
@@
 	)
 	(segment
-		(start 77.575 75.8)
-		(end 77.575 77.425)
-		(width 0.2)
-		(layer "B.Cu")
-		(net 13)
-	)
-	(segment
 		(start 85.75 72.05)
 		(end 86.55 72.05)
@@
 		(width 0.2)
 		(layer "B.Cu")
-		(net 13)
-	)
-	(segment
-		(start 77.575 77.425)
-		(end 77.525 77.475)
-		(width 0.2)
-		(layer "B.Cu")

Commit message: Finish routing for rev 1
Parts:
- removed J3: TSW-110-07-F-D, project_footprints:TSW-110-XX-YY-D
- removed SW1: SW_Push_Dual, Button_Switch_THT:SW_PUSH_6mm
- added SW2: SW_Push, Button_Switch_THT:SW_PUSH_6mm, F.Cu at (65.3, 56.0)
- moved J2 35.5 mm to (67.8, 86.3)
- moved R5 29.2 mm to (74.8, 63.3), turned to 90 degrees
- moved C10 2.80 mm to (74.4, 75.3)
Connections:
- C1 pad 1: Net-(IC1-(INT.6/AIN0)_PE6) -> Net-(IC1-PB5_(PCINT5/OC1A/~{OC4B}/ADC))
- C2 pad 1: Net-(IC1-PB5_(PCINT5/OC1A/~{OC4B}/ADC)) -> Net-(IC1-PB6_(PCINT6/OC1B/OC4B/ADC))
- C3 pad 1: Net-(IC1-(SDA/INT1)_PD1) -> Net-(IC1-(SS/PCINT0)_PB0)
- C4 pad 1: Net-(VR2-B) -> Net-(IC1-(PCINT1/SCLK)_PB1)
- IC1 pad 1: Net-(IC1-(INT.6/AIN0)_PE6) -> unconnected-(IC1-(INT.6/AIN0)_PE6-Pad1)
- IC1 pad 11: Net-(IC1-(PDO/PCINT3/MISO)_PB3) -> unconnected-(IC1-(PDO/PCINT3/MISO)_PB3-Pad11)
- IC1 pad 12: Net-(IC1-(PCINT7/OC0A/OC1C/~{RTS})_PB7) -> unconnected-(IC1-(PCINT7/OC0A/OC1C/~{RTS})_PB7-Pad12)
- IC1 pad 18: Net-(IC1-(OC0B/SCL/INT0)_PD0) -> unconnected-(IC1-(OC0B/SCL/INT0)_PD0-Pad18)
- IC1 pad 19: Net-(IC1-(SDA/INT1)_PD1) -> unconnected-(IC1-(SDA/INT1)_PD1-Pad19)
- IC1 pad 20: Net-(IC1-(RXD1/INT2)_PD2) -> unconnected-(IC1-(RXD1/INT2)_PD2-Pad20)
- IC1 pad 21: Net-(IC1-(TXD1/INT3)_PD3) -> unconnected-(IC1-(TXD1/INT3)_PD3-Pad21)
- IC1 pad 22: Net-(IC1-(XCK1/~{CTS})_PD5) -> unconnected-(IC1-(XCK1/~{CTS})_PD5-Pad22)
- IC1 pad 25: Net-(IC1-(PDI/PCINT2/MOSI)_PB2) -> unconnected-(IC1-PD4_(ICP1/ADC8)-Pad25)
- IC1 pad 26: Net-(IC1-PD6_(T1/~{OC4D}/ADC9)) -> unconnected-(IC1-PD6_(T1/~{OC4D}/ADC9)-Pad26)
- IC1 pad 27: Net-(IC1-PD7_(T0/OC4D/ADC10)) -> unconnected-(IC1-PD7_(T0/OC4D/ADC10)-Pad27)
- IC1 pad 31: Net-(IC1-PC6_(OC3A/~{OC4A})) -> unconnected-(IC1-PC6_(OC3A/~{OC4A})-Pad31)
- IC1 pad 32: Net-(IC1-PC7_(ICP3/CLK0/OC)4A) -> unconnected-(IC1-PC7_(ICP3/CLK0/OC)4A-Pad32)
- IC1 pad 33: Net-(IC1-PE2_(~{HWB})) -> unconnected-(IC1-PE2_(~{HWB})-Pad33)
- VR1 pad 1: Net-(IC1-(PCINT7/OC0A/OC1C/~{RTS})_PB7) -> Net-(IC1-PB4_(PCINT4/ADC11))
- VR1 pad A1: Net-(IC1-(INT.6/AIN0)_PE6) -> Net-(IC1-PB5_(PCINT5/OC1A/~{OC4B}/ADC))
- VR1 pad B1: Net-(IC1-PB5_(PCINT5/OC1A/~{OC4B}/ADC)) -> Net-(IC1-PB6_(PCINT6/OC1B/OC4B/ADC))
- VR2 pad 1: Net-(IC1-PB6_(PCINT6/OC1B/OC4B/ADC)) -> Net-(IC1-(PDI/PCINT2/MOSI)_PB2)
- VR2 pad A1: Net-(IC1-(SDA/INT1)_PD1) -> Net-(IC1-(SS/PCINT0)_PB0)
- VR2 pad B1: Net-(VR2-B) -> Net-(IC1-(PCINT1/SCLK)_PB1)
Routing:
- net /5V: track 60.1 -> 128.0 mm
- net Net-(IC1-~{RESET}): track 0.00 -> 49.0 mm, vias 0 -> 1
- net Net-(IC1-PB5_(PCINT5/OC1A/~{OC4B}/ADC)): track 0.00 -> 34.7 mm
- net Net-(IC1-(PCINT1/SCLK)_PB1): track 0.00 -> 33.4 mm
- net Net-(IC1-PB4_(PCINT4/ADC11)): track 0.00 -> 31.2 mm
- net Net-(IC1-PB6_(PCINT6/OC1B/OC4B/ADC)): track 0.00 -> 29.4 mm
- net Net-(IC1-(SS/PCINT0)_PB0): track 0.00 -> 28.1 mm
- net GND: track 0.00 -> 26.4 mm, vias 0 -> 3
- net Net-(IC1-PF4_(ADC4/TCK)): track 0.00 -> 23.0 mm
- net Net-(IC1-PF6_(ADC6/TDO)): track 0.00 -> 22.8 mm
- net Net-(IC1-(PDI/PCINT2/MOSI)_PB2): track 0.00 -> 22.4 mm
- net Net-(IC1-PF5_(ADC5/TMS)): track 0.00 -> 17.6 mm
- net Net-(IC1-PF7_(ADC7/TDI)): track 0.00 -> 14.7 mm
- net Net-(IC1-PE2_(~{HWB})): track 14.6 -> 0.00 mm
- net Net-(IC1-PC7_(ICP3/CLK0/OC)4A): track 13.9 -> 0.00 mm
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- added copper zone on B.Cu, net GND
- added copper zone on F.Cu, net GND
Other:
- board text added: "uhsynth scrollwheel peripheral rev 1"
- board text removed: "uhsynth scrollwheel peripheral v0.1"
